File: microcontroller/hardware/kicad/stm32Logger.sch (KiCad schematic (older format))
At the start: 35 parts

Commit message: Adding pin for one more serial RX
Parts:
- added P4: CONN_01X04, Connectors_Molex:Molex_KK-6410-04_04x2.54mm_Straight, symbol stm32Logger-rescue:CONN_01X04
- BT1: renamed from BT?; symbol Battery_Cell -> device1:Battery_Cell
- C1, C2, C3, C4, C5, C6, C7, C8, C9: renamed from C?; footprint (none) -> Capacitors_SMD:C_0603_HandSoldering; symbol C -> device1:C
- CON1: renamed from CON?; symbol Micro_SD_Card -> stm32Logger-rescue:Micro_SD_Card
- D1: renamed from D?; footprint (none) -> LEDs:LED_D3.0mm; symbol D_Photo -> device1:D_Photo
- D2, D3: renamed from D?; footprint (none) -> LEDs:LED_0603_HandSoldering; symbol LED -> device1:LED
- P1: renamed from P?; footprint (none) -> Connectors_Molex:Molex_KK-6410-03_03x2.54mm_Straight; symbol CONN_02X03 -> stm32Logger-rescue:CONN_02X03
- P2, P7: renamed from P?; footprint (none) -> Connectors_Molex:Molex_KK-6410-04_04x2.54mm_Straight; symbol CONN_01X04 -> stm32Logger-rescue:CONN_01X04
- P3, P5: renamed from P?; footprint (none) -> Connectors_Molex:Molex_KK-6410-02_02x2.54mm_Straight; symbol CONN_01X02 -> stm32Logger-rescue:CONN_01X02
- P6: renamed from P?; footprint (none) -> Connectors:USB_Micro-B; symbol USB_OTG -> stm32Logger-rescue:USB_OTG
- R1, R2, R3, R4, R5, R6, R7, R8, R9: renamed from R?; footprint (none) -> Resistors_SMD:R_0603_HandSoldering; symbol R -> device1:R
- U1: renamed from U?; symbol 74HC14 -> stm32Logger-rescue:74HC14
- U2: renamed from U?; footprint LQFP48 -> (none); symbol STM32F103C8Tx -> stm32Logger-rescue:STM32F103C8Tx
- U3: renamed from U?; symbol AP111733 -> stm32Logger-rescue:AP111733
- Y1, Y2: renamed from Y?; symbol Crystal -> device1:Crystal
Connections:
- net +3V3: now also P4.1 (P1)
- net GND: now also P4.4 (P4)
- net MeterSerial: now also P4.3 (P3)
- net Serial2RX: now reaches U2.13 (ADC1_IN3/ADC2_IN3/TIM2_CH4/USART2_RX/PA3)
- net Serial2RX: now also P4.2 (P2)
